File: usblink.brd (EAGLE design)
At the start: 37.8 x 38.1 mm, 20 parts, among them T1 2N2222, T2 2N2222

Commit message: Add files via upload
Parts:
- removed R6: 1k, pot:B25V
- added R5: 1k, pot:3RP/1610N
- moved T1 11.4 mm to (33.0, 21.6)
- moved _D 11.4 mm to (26.7, 3.81)
- moved C2 11.4 mm to (34.3, 10.2)
- moved C3 11.4 mm to (31.8, 27.9)
- moved D3 11.4 mm to (19.1, 25.4)
- moved R1 11.4 mm to (38.1, 24.1)
- moved R2 11.4 mm to (40.6, 34.3)
- moved R3 11.4 mm to (14.0, 25.4)
- moved T2 11.4 mm to (19.1, 16.5)
- moved _+ 11.4 mm to (34.3, 3.81)
- moved _A 11.4 mm to (29.2, 3.81)
- moved _B 11.4 mm to (31.8, 3.81)
- moved _G 11.4 mm to (24.1, 3.81)
- moved C4 11.4 mm to (25.4, 24.1)
- moved D1 11.4 mm to (25.4, 35.6)
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Connections:
- net DATA: now also R5.2; no longer R6.S
- net GND: now also R5.1; no longer R6.A
- net N$4: now also R5.3; no longer R6.E
Routing:
- net DATA: track 10.2 -> 17.3 mm
- net N$4: track 15.1 -> 18.2 mm
- net GND: track 59.6 -> 60.5 mm
Other:
- board size 37.8 x 38.1 mm -> 49.2 x 38.1 mm
- board text added: "JAKE-LINK"
- board text removed: "USB-LINK"
