File: usblink.sch (EAGLE design)
At the start: 20 parts, among them T1 2N2222, T2 2N2222

Commit message: Add files via upload
Parts:
- removed R6: 1k, pot:TRIM_US-B25V
- added R5: 1k, pot:3RP/1610N
Connections:
- net DATA: now also R5.S; no longer R6.S
- net GND: now also R5.A; no longer R6.A
- net N$4: now also R5.E; no longer R6.E
Changed lines of the file:
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@@
 <part name="R4" library="adafruit" deviceset="R-US_" device="0204/7" value="330k"/>
 <part name="S1" library="adafruit" deviceset="EG1218" device="S"/>
-<part name="R6" library="pot" deviceset="TRIM_US-" device="B25V" value="1k"/>
 <part name="GND1" library="supply1" deviceset="GND" device=""/>
 <part name="GND2" library="supply1" deviceset="GND" device=""/>
@@
 <part name="_G" library="adafruit" deviceset="PINHD-1X1" device="CB"/>
 <part name="_B" library="adafruit" deviceset="PINHD-1X1" device="CB"/>
+<part name="R5" library="pot" deviceset="3RP/1610N" device="" value="1k"/>
 </parts>
 <sheets>
@@
 <instance part="R4" gate="G$1" x="27.94" y="43.18" rot="R180"/>
 <instance part="S1" gate="1" x="5.08" y="81.28" rot="R270"/>
-<instance part="R6" gate="G$1" x="20.32" y="60.96"/>
 <instance part="GND1" gate="1" x="119.38" y="10.16"/>
 <instance part="GND2" gate="1" x="-12.7" y="10.16"/>
@@
 <instance part="_G" gate="G$1" x="-15.24" y="12.7" rot="R180"/>
 <instance part="_B" gate="G$1" x="121.92" y="22.86"/>
+<instance part="R5" gate="G$1" x="20.32" y="60.96"/>
 </instances>
 <busses>
@@
 <segment>
 <pinref part="C2" gate="G$1" pin="1"/>
-<pinref part="R6" gate="G$1" pin="E"/>
 <wire x1="15.24" y1="68.58" x2="20.32" y2="68.58" width="0.1524" layer="91"/>
 <junction x="15.24" y="68.58"/>
-<junction x="20.32" y="68.58"/>
+<pinref part="R5" gate="G$1" pin="E"/>
+<wire x1="20.32" y1="68.58" x2="20.32" y2="66.04" width="0.1524" layer="91"/>
 </segment>
 </net>
@@
 <junction x="33.02" y="22.86"/>
 <junction x="33.02" y="12.7"/>
-<pinref part="R6" gate="G$1" pin="A"/>
-<wire x1="20.32" y1="53.34" x2="20.32" y2="12.7" width="0.1524" layer="91"/>
+<wire x1="20.32" y1="55.88" x2="20.32" y2="12.7" width="0.1524" layer="91"/>
 <junction x="20.32" y="12.7"/>
-<junction x="20.32" y="53.34"/>
 <label x="-7.62" y="12.7" size="1.778" layer="95"/>
 <label x="116.84" y="12.7" size="1.778" layer="95" rot="R180"/>
@@
 <pinref part="GND2" gate="1" pin="GND"/>
 <pinref part="_G" gate="G$1" pin="1"/>
+<pinref part="R5" gate="G$1" pin="A"/>
+<junction x="20.32" y="55.88"/>
 </segment>
 </net>
 <net name="DATA" class="0">
 <segment>
-<pinref part="R6" gate="G$1" pin="S"/>
 <wire x1="25.4" y1="60.96" x2="50.8" y2="60.96" width="0.1524" layer="91"/>
-<junction x="25.4" y="60.96"/>
 <label x="43.18" y="60.96" size="1.778" layer="95"/>
 <pinref part="_D" gate="G$1" pin="1"/>
-</segment>
-</net>
+<pinref part="R5" gate="G$1" pin="S"/>
+<junction x="25.4" y="60.96"/>
+</segment>
+</net>
